File: Mother_STM32F411_Disco.kicad_pcb (KiCad board)
At the start: 2 copper layers, 2 parts

Commit message: Huellas y netlist
Parts:
- added 1_Out_Ampl1: Conn_01x02, Connector_PinSocket_2.54mm:PinSocket_1x02_P2.54mm_Vertical, F.Cu at (210.5, 14.8)
- added 1_Out_Ampl2: Conn_01x02, Connector_PinSocket_2.54mm:PinSocket_1x02_P2.54mm_Vertical, F.Cu at (221.0, 29.2)
- added 1_Out_Ampl3: Conn_01x02, Connector_PinSocket_2.54mm:PinSocket_1x02_P2.54mm_Vertical, F.Cu at (257.0, 15.2)
- added 2_Out_Ampl1: Conn_01x02, Connector_PinSocket_2.54mm:PinSocket_1x02_P2.54mm_Vertical, F.Cu at (211.0, 28.2)
- added 2_Out_Ampl2: Conn_01x02, Connector_PinSocket_2.54mm:PinSocket_1x02_P2.54mm_Vertical, F.Cu at (233.0, 29.5)
- added 2_Out_Ampl3: Conn_01x02, Connector_PinSocket_2.54mm:PinSocket_1x02_P2.54mm_Vertical, F.Cu at (257.0, 29.5)
- added Audio_IN_Ampl1: Conn_01x03, Connector_PinSocket_2.54mm:PinSocket_1x03_P2.54mm_Vertical, F.Cu at (227.3, 42.5)
- added Audio_IN_Ampl2: Conn_01x03, Connector_PinSocket_2.54mm:PinSocket_1x03_P2.54mm_Vertical, F.Cu at (220.5, 15.5)
- added Audio_IN_Ampl3: Conn_01x03, Connector_PinSocket_2.54mm:PinSocket_1x03_P2.54mm_Vertical, F.Cu at (244.0, 26.5)
- added Multiplex_Audio_in1: Conn_02x08_Counter_Clockwise, Connector_PinSocket_2.54mm:PinSocket_2x08_P2.54mm_Vertical, F.Cu at (172.0, 96.5)
- added Multiplex_Audio_out_1: Conn_01x03, Connector_PinSocket_2.54mm:PinSocket_1x03_P2.54mm_Vertical, F.Cu at (205.0, 73.0)
- added Multiplex_Audio_out_2: Conn_01x03, Connector_PinSocket_2.54mm:PinSocket_1x03_P2.54mm_Vertical, F.Cu at (204.4, 98.5)
- added Multiplex_Audio_out_3: Conn_01x03, Connector_PinSocket_2.54mm:PinSocket_1x03_P2.54mm_Vertical, F.Cu at (204.5, 107.0)
- added Out_Speaker_1: Conn_01x02, Connector_PinHeader_2.54mm:PinHeader_1x02_P2.54mm_Horizontal, F.Cu at (263.8, 64.9)
- added Out_Speaker_2: Conn_01x02, Connector_PinHeader_2.54mm:PinHeader_1x02_P2.54mm_Horizontal, F.Cu at (265.1, 74.2)
- added Out_Speaker_3: Conn_01x02, Connector_PinHeader_2.54mm:PinHeader_1x02_P2.54mm_Horizontal, F.Cu at (265.1, 81.4)
- added Out_Speaker_4: Conn_01x02, Connector_PinHeader_2.54mm:PinHeader_1x02_P2.54mm_Horizontal, F.Cu at (265.1, 88.5)
- added Out_Speaker_5: Conn_01x02, Connector_PinHeader_2.54mm:PinHeader_1x02_P2.54mm_Horizontal, F.Cu at (265.1, 95.6)
- added Out_Speaker_6: Conn_01x02, Connector_PinHeader_2.54mm:PinHeader_1x02_P2.54mm_Horizontal, F.Cu at (265.1, 102.8)
- added PWR_Ampl1: Conn_01x02, Connector_PinSocket_2.54mm:PinSocket_1x02_P2.54mm_Vertical, F.Cu at (227.3, 55.1)
- added PWR_Ampl2: Conn_01x02, Connector_PinSocket_2.54mm:PinSocket_1x02_P2.54mm_Vertical, F.Cu at (227.0, 22.2)
- added PWR_Ampl3: Conn_01x02, Connector_PinSocket_2.54mm:PinSocket_1x02_P2.54mm_Vertical, F.Cu at (250.0, 23.5)
- added Pantalla-Botones1: Conn_01x08, Connector_PinSocket_2.54mm:PinSocket_1x08_P2.54mm_Vertical, F.Cu at (35.5, 30.9)
- moved Conn_Der_STM_Disco1 31.6 mm to (134.5, 58.6)
- moved Conn_Izq_STM_Disco1 21.4 mm to (75.0, 58.5)
Other:
- board text added: "AMPL_1 PAM8403"
