File: Mother_STM32F411_Disco.kicad_pcb (KiCad board)
At the start: 2 copper layers, 25 parts

Commit message: Huellas prearmadas, falta comprobar medidas
Parts:
- moved Pantalla-Botones1 171.9 mm to (165.1, 143.8)
- moved Multiplex_Audio_out_3 99.9 mm to (120.5, 53.0)
- moved Multiplex_Audio_in1 99.9 mm to (88.0, 42.5)
- moved Multiplex_Audio_out_1 99.9 mm to (121.0, 19.0)
- moved Multiplex_Audio_out_2 99.9 mm to (120.4, 44.5)
- moved Conn_Der_STM_Disco1 78.5 mm to (59.9, 34.2)
- moved Conn_Izq_STM_Disco1 71.3 mm to (8.00, 34.1)
- moved Audio_IN_Ampl1 53.0 mm to (179.2, 20.3)
- moved PWR_Ampl1 53.0 mm to (179.2, 32.9)
- moved Out_Speaker_2 26.4 mm to (239.3, 68.4)
- moved Out_Speaker_3 26.4 mm to (239.3, 75.5)
- moved Out_Speaker_4 26.4 mm to (239.3, 82.6)
- moved Out_Speaker_5 26.4 mm to (239.3, 89.8)
- moved Out_Speaker_6 26.4 mm to (239.3, 96.9)
- moved Out_Speaker_1 26.4 mm to (238.0, 59.0)
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- renumbered 1_Out_Ampl1 to 1_Out, 2_Out_Ampl1 to 2_Out, 2_Out_Ampl3 to Out, 1_Out_Ampl2 to Out, 1_Out_Ampl3 to Out, 2_Out_Ampl2 to Out
Other:
- board text added: "AMPL_2 PAM8403"
- board text added: "AMPL_3 PAM8403"
- board text removed: "Amplificador"
